Commit message: ekf initial build

File: CODE/ros_ws/src/localization/urdf/robot.urdf.xacro (robot description, xacro)
@@ -2,17 +2,15 @@
 <!--
   robot.urdf.xacro
-  TF Tree (ZED-rooted, no odom_base_publisher):
-    map → odom → zed_left_camera_frame → zed_camera_link → base_link → left_wheel
-                                        → zed_imu_link              → right_wheel
-                                        → zed_right_camera_frame
-                                        → zed_camera_center
-                                        → (other ZED internal frames)
+  TF Tree (EKF-owned):
+    map → odom → base_link → zed_camera_link → zed_camera_center → zed_left_camera_frame
+                           ├── left_wheel             → zed_right_camera_frame
+                           ├── right_wheel            → zed_imu_link
+                           └── ground                 → (other ZED internal frames)
   Frame convention:
-    - zed_camera_link is the ZED's gravity-aligned root (two_d_mode + set_gravity_as_origin)
-    - base_link hangs off zed_camera_link, offset back and down to ground level
-    - No tilt in the joint — ZED gravity alignment already levels the frame
-    - Wheel visuals are children of base_link as before
-  ZED config: publish_tf: true, two_d_mode: true, set_gravity_as_origin: true
-  No odom_base_publisher needed — ZED owns map→odom→zed_left_camera_frame→zed_camera_link
+    - base_link is the robot body root (EKF publishes odom→base_link)
+    - zed_camera_link is a child of base_link via static_transform_publisher
+      (in robot_description.launch.py: xyz=0.174 0 -0.05, rpy=0 0 0)
+    - ZED SDK publishes its internal camera frames as children of zed_camera_link via /tf_static
+    - ZED config: publish_tf: false (EKF owns the TF chain)
 -->
 <robot xmlns:xacro="http://www.ros.org/wiki/xacro" name="material_transfer_robot">
@@ -26,7 +24,12 @@
   <xacro:property name="wheel_width" value="0.026"/>
   <xacro:property name="wheel_y_offset" value="0.063"/>
-  <!-- ZED CAMERA LINK — root of URDF tree, owned by ZED SDK TF broadcaster -->
-  <!-- Declared here so robot_state_publisher knows it exists as a root -->
+  <!-- ZED CAMERA LINK — child of base_link, forward and down from robot center -->
   <link name="zed_camera_link"/>
+  <joint name="base_to_camera_joint" type="fixed">
+    <parent link="base_link"/>
+    <child link="zed_camera_link"/>
+    <!-- Inverse of old camera_to_base_joint: +forward, -up -->
+    <origin xyz="${camera_forward} 0 ${-wheel_radius}" rpy="0 0 0"/>
+  </joint>
   <!-- Camera mount frame: true physical pose (height + tilt) -->
   <link name="camera_mount"/>
@@ -36,11 +39,4 @@
     <!-- Raise by camera_height and apply tilt (no forward offset here) -->
     <origin xyz="0 0 ${camera_height}" rpy="0 ${camera_tilt} 0"/>
-  </joint>
-  <!-- BASE LINK — upright, at robot center, raised by wheel_radius -->
-  <joint name="camera_to_base_joint" type="fixed">
-    <parent link="zed_camera_link"/>
-    <child link="base_link"/>
-    <!-- zed_camera_link is at ground, base_link at wheel_radius above ground -->
-    <origin xyz="${-camera_forward} 0 ${wheel_radius}" rpy="0 0 0"/>
   </joint>
   <!-- Ground frame at floor level -->

Commit message: fix: camera tilt angle

File: CODE/ros_ws/src/localization/urdf/robot.urdf.xacro (robot description, xacro)
@@ -20,5 +20,5 @@
   <xacro:property name="camera_height" value="0.746"/>
   <xacro:property name="camera_forward" value="0.174"/>
-  <xacro:property name="camera_tilt" value="-0.5236"/>
+  <xacro:property name="camera_tilt" value="0.5236"/>
   <xacro:property name="wheel_radius" value="0.05"/>
   <xacro:property name="wheel_width" value="0.026"/>
@@ -34,9 +34,9 @@
   <!-- Camera mount frame: true physical pose (height + tilt) -->
   <link name="camera_mount"/>
-  <joint name="zed_to_camera_mount" type="fixed">
-    <parent link="zed_camera_link"/>
+  <joint name="base_to_camera_mount" type="fixed">
+    <parent link="base_link"/>
     <child link="camera_mount"/>
     <!-- Raise by camera_height and apply tilt (no forward offset here) -->
-    <origin xyz="0 0 ${camera_height}" rpy="0 ${camera_tilt} 0"/>
+    <origin xyz="${camera_forward} 0 ${camera_height}" rpy="0 ${camera_tilt} 0"/>
   </joint>
   <!-- Ground frame at floor level -->
