Commit message: fix base_link to odom frame link

File: CODE/ros_ws/src/robot_bringup/urdf/robot.urdf.xacro (robot description, xacro)
@@ -2,112 +2,91 @@
 <!--
   robot.urdf.xacro
-  Simple URDF for physical robot with ZED Mini camera
-  IMPORTANT: Measure and update the camera position to match YOUR robot!
-  Coordinate system (REP 103):
-    x = forward (red axis in RViz)
-    y = left (green axis in RViz)
-    z = up (blue axis in RViz)
-  Place this file in: robot_bringup/urdf/robot.urdf.xacro
+  TF Tree after this URDF + ZED:
+    map → odom → zed_camera_link → base_link → wheels
+    (ZED)  (ZED)     (ZED)           (URDF)     (URDF)
+  ZED publishes: map → odom → zed_camera_link
+  URDF publishes: zed_camera_link → base_link → wheels
 -->
 <robot xmlns:xacro="http://www.ros.org/wiki/xacro" name="material_transfer_robot">
   <!-- ============================================ -->
-  <!-- ROBOT PARAMETERS - MEASURE AND UPDATE THESE -->
+  <!-- ROBOT PARAMETERS                            -->
   <!-- ============================================ -->
-  <!-- Robot body dimensions (meters) -->
-  <xacro:property name="body_length" value="0.40" />
-  <!-- Front to back -->
-  <xacro:property name="body_width" value="0.40" />
-  <!-- Left to right -->
-  <xacro:property name="body_height" value="0.15" />
-  <!-- Height of body -->
-  <!-- Camera mount position relative to base_link center -->
-  <!-- MEASURE THESE ON YOUR PHYSICAL ROBOT! -->
-  <xacro:property name="camera_x" value="0.10" />
-  <!-- Forward from center -->
-  <xacro:property name="camera_y" value="0.00" />
-  <!-- Left from center (0 = centered) -->
-  <xacro:property name="camera_z" value="0.25" />
-  <!-- Height above ground -->
-  <!-- Camera rotation (radians) - usually 0 if camera faces forward -->
-  <xacro:property name="camera_roll" value="0.0" />
-  <xacro:property name="camera_pitch" value="0.523" />
-  <xacro:property name="camera_yaw" value="0.0" />
+  <!-- Robot body dimensions (meters) - for visualization -->
+  <xacro:property name="body_length" value="0.40"/>
+  <xacro:property name="body_width" value="0.40"/>
+  <xacro:property name="body_height" value="0.70"/>
+  <!-- Camera to base_link offset (zed_camera_link → base_link) -->
+  <!-- These match your original static_transform_publisher values -->
+  <xacro:property name="base_x" value="-0.15"/>     <!-- base_link is 15cm BEHIND camera -->
+  <xacro:property name="base_y" value="0.00"/>      <!-- Centered -->
+  <xacro:property name="base_z" value="-0.70"/>     <!-- base_link is 70cm BELOW camera -->
+  <!-- Camera rotation relative to base -->
+  <xacro:property name="base_roll" value="0.0"/>
+  <xacro:property name="base_pitch" value="-0.523"/>  <!-- -30° (camera tilted down) -->
+  <xacro:property name="base_yaw" value="0.0"/>
+  <!-- Wheel parameters -->
+  <xacro:property name="wheel_radius" value="0.05"/>
+  <xacro:property name="wheel_width" value="0.04"/>
+  <xacro:property name="wheel_y_offset" value="0.20"/>
   <!-- ============================================ -->
-  <!-- BASE LINK - Robot center/footprint          -->
+  <!-- ZED CAMERA LINK (root of URDF, child of odom via ZED) -->
   <!-- ============================================ -->
+  <link name="zed_camera_link"/>
+  <!-- ============================================ -->
+  <!-- BASE LINK - Connected to camera             -->
+  <!-- ============================================ -->
+  <joint name="camera_to_base_joint" type="fixed">
+    <parent link="zed_camera_link"/>
+    <child link="base_link"/>
+    <origin xyz="${base_x} ${base_y} ${base_z}"
+            rpy="${base_roll} ${base_pitch} ${base_yaw}"/>
+  </joint>
   <link name="base_link">
     <visual>
       <geometry>
-        <box size="${body_length} ${body_width} ${body_height}" />
+        <box size="${body_length} ${body_width} ${body_height}"/>
       </geometry>
-      <origin xyz="0 0 ${body_height/2}" rpy="0 0 0" />
+      <origin xyz="0 0 ${body_height/2}" rpy="0 0 0"/>
       <material name="grey">
-        <color rgba="0.5 0.5 0.5 1" />
+        <color rgba="0.5 0.5 0.5 1"/>
       </material>
     </visual>
     <collision>
       <geometry>
-        <box size="${body_length} ${body_width} ${body_height}" />
+        <box size="${body_length} ${body_width} ${body_height}"/>
       </geometry>
-      <origin xyz="0 0 ${body_height/2}" rpy="0 0 0" />
+      <origin xyz="0 0 ${body_height/2}" rpy="0 0 0"/>
     </collision>
   </link>
   <!-- ============================================ -->
-  <!-- ZED CAMERA MOUNT                            -->
+  <!-- WHEELS                                      -->
   <!-- ============================================ -->
-  <!--
-    This joint defines the STATIC transform: zed_camera_link → base_link
-    robot_state_publisher will broadcast this TF
-  -->
-  <joint name="zed_camera_joint" type="fixed">
-    <parent link="base_link" />
-    <child link="zed_camera_link" />
-    <origin xyz="${camera_x} ${camera_y} ${camera_z}"
-      rpy="${camera_roll} ${camera_pitch} ${camera_yaw}" />
-  </joint>
-  <link name="zed_camera_link">
-    <visual>
-      <geometry>
-        <!-- ZED Mini approximate dimensions -->
-        <box size="0.03 0.175 0.03" />
-      </geometry>
-      <material name="dark_grey">
-        <color rgba="0.2 0.2 0.2 1" />
-      </material>
-    </visual>
-  </link>
-  <!-- ============================================ -->
-  <!-- OPTIONAL: Wheels (for visualization only)   -->
-  <!-- ============================================ -->
-  <xacro:property name="wheel_radius" value="0.05" />
-  <xacro:property name="wheel_width" value="0.04" />
-  <xacro:property name="wheel_y_offset" value="0.20" />
   <joint name="left_wheel_joint" type="fixed">
-    <parent link="base_link" />
-    <child link="left_wheel" />
-    <origin xyz="0 ${wheel_y_offset} ${wheel_radius}" rpy="-1.5708 0 0" />
+    <parent link="base_link"/>
+    <child link="left_wheel"/>
+    <origin xyz="0 ${wheel_y_offset} ${wheel_radius}" rpy="-1.5708 0 0"/>
   </joint>
   <link name="left_wheel">
     <visual>
       <geometry>
-        <cylinder radius="${wheel_radius}" length="${wheel_width}" />
+        <cylinder radius="${wheel_radius}" length="${wheel_width}"/>
       </geometry>
       <material name="black">
-        <color rgba="0.1 0.1 0.1 1" />
+        <color rgba="0.1 0.1 0.1 1"/>
       </material>
     </visual>
   </link>
   <joint name="right_wheel_joint" type="fixed">
-    <parent link="base_link" />
-    <child link="right_wheel" />
-    <origin xyz="0 -${wheel_y_offset} ${wheel_radius}" rpy="-1.5708 0 0" />
+    <parent link="base_link"/>
+    <child link="right_wheel"/>
+    <origin xyz="0 -${wheel_y_offset} ${wheel_radius}" rpy="-1.5708 0 0"/>
   </joint>
   <link name="right_wheel">
     <visual>
       <geometry>
-        <cylinder radius="${wheel_radius}" length="${wheel_width}" />
+        <cylinder radius="${wheel_radius}" length="${wheel_width}"/>
       </geometry>
       <material name="black">
-        <color rgba="0.1 0.1 0.1 1" />
+        <color rgba="0.1 0.1 0.1 1"/>
       </material>
     </visual>

Commit message: fix wheel positions w.r.t base link

File: CODE/ros_ws/src/robot_bringup/urdf/robot.urdf.xacro (robot description, xacro)
@@ -2,9 +2,22 @@
 <!--
   robot.urdf.xacro
-  TF Tree after this URDF + ZED:
+  TF Tree:
     map → odom → zed_camera_link → base_link → wheels
     (ZED)  (ZED)     (ZED)           (URDF)     (URDF)
-  ZED publishes: map → odom → zed_camera_link
-  URDF publishes: zed_camera_link → base_link → wheels
+  Camera mounting (in WORLD/base_link frame, before rotation):
+    - Camera is 0.746m directly ABOVE base_link (Z axis)
+    - Camera is 0.174m FORWARD of base_link center (X axis)
+    - Camera is THEN tilted 30° down (pitch rotation)
+  To get base_link position in zed_camera_link frame:
+    1. Start at camera position
+    2. Apply INVERSE of camera pose
+  Since camera is tilted 30° down, its Z axis points 30° below horizontal.
+  base_link is behind and below in camera's rotated frame.
+  Transform: zed_camera_link → base_link
+    Position (in camera's tilted frame):
+      x = -forward * cos(tilt) + height * sin(tilt)  (behind camera)
+      z = -forward * sin(tilt) - height * cos(tilt)  (below camera)
+    Rotation:
+      pitch = +tilt (counter-rotate so base_link is level)
 -->
 <robot xmlns:xacro="http://www.ros.org/wiki/xacro" name="material_transfer_robot">
@@ -12,81 +25,95 @@
   <!-- ROBOT PARAMETERS                            -->
   <!-- ============================================ -->
-  <!-- Robot body dimensions (meters) - for visualization -->
-  <xacro:property name="body_length" value="0.40"/>
-  <xacro:property name="body_width" value="0.40"/>
-  <xacro:property name="body_height" value="0.70"/>
-  <!-- Camera to base_link offset (zed_camera_link → base_link) -->
-  <!-- These match your original static_transform_publisher values -->
-  <xacro:property name="base_x" value="-0.15"/>     <!-- base_link is 15cm BEHIND camera -->
-  <xacro:property name="base_y" value="0.00"/>      <!-- Centered -->
-  <xacro:property name="base_z" value="-0.70"/>     <!-- base_link is 70cm BELOW camera -->
-  <!-- Camera rotation relative to base -->
-  <xacro:property name="base_roll" value="0.0"/>
-  <xacro:property name="base_pitch" value="-0.523"/>  <!-- -30° (camera tilted down) -->
-  <xacro:property name="base_yaw" value="0.0"/>
+  <!-- Robot body dimensions (meters) -->
+  <xacro:property name="body_length" value="0.40" />
+  <xacro:property name="body_width" value="0.30" />
+  <xacro:property name="body_height" value="0.70" />
+  <!-- Camera mount (measured in world frame, camera level) -->
+  <xacro:property name="camera_height" value="0.746" />
+  <!-- Vertical height above base_link -->
+  <xacro:property name="camera_forward" value="0.174" />
+  <!-- Forward of base_link center -->
+  <xacro:property name="camera_tilt" value="0.523" />
+  <!-- 30° down tilt in radians -->
+  <!-- Transform: zed_camera_link → base_link -->
+  <!-- base_link position in camera's tilted coordinate frame -->
+  <xacro:property name="base_x"
+    value="${-camera_forward * cos(camera_tilt) + camera_height * sin(camera_tilt)}" />
+  <xacro:property name="base_y" value="0.0" />
+  <xacro:property name="base_z"
+    value="${-camera_forward * sin(camera_tilt) - camera_height * cos(camera_tilt)}" />
   <!-- Wheel parameters -->
-  <xacro:property name="wheel_radius" value="0.05"/>
-  <xacro:property name="wheel_width" value="0.04"/>
-  <xacro:property name="wheel_y_offset" value="0.20"/>
+  <xacro:property name="wheel_radius" value="0.075" />
+  <!-- 7.5cm radius -->
+  <xacro:property name="wheel_width" value="0.026" />
+  <!-- 4cm wide -->
+  <xacro:property name="wheel_y_offset" value="0.063" />
+  <!-- Distance from center to wheel -->
   <!-- ============================================ -->
-  <!-- ZED CAMERA LINK (root of URDF, child of odom via ZED) -->
+  <!-- ZED CAMERA LINK (published by ZED SDK)      -->
   <!-- ============================================ -->
-  <link name="zed_camera_link"/>
+  <link name="zed_camera_link" />
   <!-- ============================================ -->
-  <!-- BASE LINK - Connected to camera             -->
+  <!-- BASE LINK - Robot center at ground level    -->
   <!-- ============================================ -->
   <joint name="camera_to_base_joint" type="fixed">
-    <parent link="zed_camera_link"/>
-    <child link="base_link"/>
-    <origin xyz="${base_x} ${base_y} ${base_z}"
-            rpy="${base_roll} ${base_pitch} ${base_yaw}"/>
+    <parent link="zed_camera_link" />
+    <child link="base_link" />
+    <!-- Position in camera frame, then rotate to level -->
+    <origin xyz="${base_x} ${base_y} ${base_z}" rpy="0 ${camera_tilt} 0" />
   </joint>
   <link name="base_link">
     <visual>
       <geometry>
-        <box size="${body_length} ${body_width} ${body_height}"/>
+        <box size="${body_length} ${body_width} ${body_height}" />
       </geometry>
-      <origin xyz="0 0 ${body_height/2}" rpy="0 0 0"/>
+      <!-- Box centered at body_height/2 so bottom is at z=0 -->
+      <origin xyz="0 0 ${body_height/2}" rpy="0 0 0" />
       <material name="grey">
-        <color rgba="0.5 0.5 0.5 1"/>
+        <color rgba="0.6 0.6 0.6 0.8" />
       </material>
     </visual>
     <collision>
       <geometry>
-        <box size="${body_length} ${body_width} ${body_height}"/>
+        <box size="${body_length} ${body_width} ${body_height}" />
       </geometry>
-      <origin xyz="0 0 ${body_height/2}" rpy="0 0 0"/>
+      <origin xyz="0 0 ${body_height/2}" rpy="0 0 0" />
     </collision>
   </link>
   <!-- ============================================ -->
-  <!-- WHEELS                                      -->
+  <!-- LEFT WHEEL                                  -->
   <!-- ============================================ -->
   <joint name="left_wheel_joint" type="fixed">
-    <parent link="base_link"/>
-    <child link="left_wheel"/>
-    <origin xyz="0 ${wheel_y_offset} ${wheel_radius}" rpy="-1.5708 0 0"/>
+    <parent link="base_link" />
+    <child link="left_wheel" />
+    <!-- Wheel at ground level (z = wheel_radius), offset to left (+y) -->
+    <origin xyz="0 ${body_width/2+wheel_y_offset} 0" rpy="${-pi/2} 0 0" />
   </joint>
   <link name="left_wheel">
     <visual>
       <geometry>
-        <cylinder radius="${wheel_radius}" length="${wheel_width}"/>
+        <cylinder radius="${wheel_radius}" length="${wheel_width}" />
       </geometry>
-      <material name="black">
-        <color rgba="0.1 0.1 0.1 1"/>
+      <material name="dark_grey">
+        <color rgba="0.2 0.2 0.2 1.0" />
       </material>
     </visual>
   </link>
+  <!-- ============================================ -->
+  <!-- RIGHT WHEEL                                 -->
+  <!-- ============================================ -->
   <joint name="right_wheel_joint" type="fixed">
-    <parent link="base_link"/>
-    <child link="right_wheel"/>
-    <origin xyz="0 -${wheel_y_offset} ${wheel_radius}" rpy="-1.5708 0 0"/>
+    <parent link="base_link" />
+    <child link="right_wheel" />
+    <!-- Wheel at ground level, offset to right (-y) -->
+    <origin xyz="0 ${-body_width/2-wheel_y_offset} 0" rpy="${-pi/2} 0 0" />
   </joint>
   <link name="right_wheel">
     <visual>
       <geometry>
-        <cylinder radius="${wheel_radius}" length="${wheel_width}"/>
+        <cylinder radius="${wheel_radius}" length="${wheel_width}" />
       </geometry>
-      <material name="black">
-        <color rgba="0.1 0.1 0.1 1"/>
+      <material name="dark_grey">
+        <color rgba="0.2 0.2 0.2 1.0" />
       </material>
     </visual>

Commit message: disable 2d mode and fix frame transformation

File: CODE/ros_ws/src/robot_bringup/urdf/robot.urdf.xacro (robot description, xacro)
@@ -30,7 +30,7 @@
   <xacro:property name="body_height" value="0.70" />
   <!-- Camera mount (measured in world frame, camera level) -->
-  <xacro:property name="camera_height" value="0.746" />
+  <xacro:property name="camera_height" value="0.75" />
   <!-- Vertical height above base_link -->
-  <xacro:property name="camera_forward" value="0.174" />
+  <xacro:property name="camera_forward" value="0.17" />
   <!-- Forward of base_link center -->
   <xacro:property name="camera_tilt" value="0.523" />
@@ -61,5 +61,5 @@
     <child link="base_link" />
     <!-- Position in camera frame, then rotate to level -->
-    <origin xyz="${base_x} ${base_y} ${base_z}" rpy="0 ${camera_tilt} 0" />
+    <origin xyz="${base_x} ${base_y} ${base_z}" rpy="0 ${-camera_tilt} 0" />
   </joint>
   <link name="base_link">

Commit message: fix frame linkage

File: CODE/ros_ws/src/robot_bringup/urdf/robot.urdf.xacro (robot description, xacro)
@@ -2,65 +2,25 @@
 <!--
   robot.urdf.xacro
-  TF Tree:
-    map → odom → zed_camera_link → base_link → wheels
-    (ZED)  (ZED)     (ZED)           (URDF)     (URDF)
-  Camera mounting (in WORLD/base_link frame, before rotation):
-    - Camera is 0.746m directly ABOVE base_link (Z axis)
-    - Camera is 0.174m FORWARD of base_link center (X axis)
-    - Camera is THEN tilted 30° down (pitch rotation)
-  To get base_link position in zed_camera_link frame:
-    1. Start at camera position
-    2. Apply INVERSE of camera pose
-  Since camera is tilted 30° down, its Z axis points 30° below horizontal.
-  base_link is behind and below in camera's rotated frame.
-  Transform: zed_camera_link → base_link
-    Position (in camera's tilted frame):
-      x = -forward * cos(tilt) + height * sin(tilt)  (behind camera)
-      z = -forward * sin(tilt) - height * cos(tilt)  (below camera)
-    Rotation:
-      pitch = +tilt (counter-rotate so base_link is level)
+  TF Tree (with odom_base_publisher node):
+    map → odom → base_link → zed_camera_link
+    (node) (node)   (URDF)
+  Camera mounting (in base_link frame):
+    - 0.746m above base_link (Z)
+    - 0.174m forward of base_link center (X)
+    - 30° nose-down tilt (pitch = 0.523 rad)
+  ZED config: publish_tf: false, publish_map_tf: false
+  odom_base_publisher handles all dynamic TFs.
 -->
 <robot xmlns:xacro="http://www.ros.org/wiki/xacro" name="material_transfer_robot">
-  <!-- ============================================ -->
-  <!-- ROBOT PARAMETERS                            -->
-  <!-- ============================================ -->
-  <!-- Robot body dimensions (meters) -->
   <xacro:property name="body_length" value="0.40" />
-  <xacro:property name="body_width" value="0.30" />
+  <xacro:property name="body_width"  value="0.30" />
   <xacro:property name="body_height" value="0.70" />
-  <!-- Camera mount (measured in world frame, camera level) -->
-  <xacro:property name="camera_height" value="0.75" />
-  <!-- Vertical height above base_link -->
-  <xacro:property name="camera_forward" value="0.17" />
-  <!-- Forward of base_link center -->
-  <xacro:property name="camera_tilt" value="0.523" />
-  <!-- 30° down tilt in radians -->
-  <!-- Transform: zed_camera_link → base_link -->
-  <!-- base_link position in camera's tilted coordinate frame -->
-  <xacro:property name="base_x"
-    value="${-camera_forward * cos(camera_tilt) + camera_height * sin(camera_tilt)}" />
-  <xacro:property name="base_y" value="0.0" />
-  <xacro:property name="base_z"
-    value="${-camera_forward * sin(camera_tilt) - camera_height * cos(camera_tilt)}" />
-  <!-- Wheel parameters -->
-  <xacro:property name="wheel_radius" value="0.075" />
-  <!-- 7.5cm radius -->
-  <xacro:property name="wheel_width" value="0.026" />
-  <!-- 4cm wide -->
+  <xacro:property name="camera_height"  value="0.746" />
+  <xacro:property name="camera_forward" value="0.174" />
+  <xacro:property name="camera_tilt"    value="0.523" />
+  <xacro:property name="wheel_radius"   value="0.075" />
+  <xacro:property name="wheel_width"    value="0.026" />
   <xacro:property name="wheel_y_offset" value="0.063" />
-  <!-- Distance from center to wheel -->
-  <!-- ============================================ -->
-  <!-- ZED CAMERA LINK (published by ZED SDK)      -->
-  <!-- ============================================ -->
-  <link name="zed_camera_link" />
-  <!-- ============================================ -->
-  <!-- BASE LINK - Robot center at ground level    -->
-  <!-- ============================================ -->
-  <joint name="camera_to_base_joint" type="fixed">
-    <parent link="zed_camera_link" />
-    <child link="base_link" />
-    <!-- Position in camera frame, then rotate to level -->
-    <origin xyz="${base_x} ${base_y} ${base_z}" rpy="0 ${-camera_tilt} 0" />
-  </joint>
+  <!-- BASE LINK -->
   <link name="base_link">
     <visual>
@@ -68,9 +28,6 @@
         <box size="${body_length} ${body_width} ${body_height}" />
       </geometry>
-      <!-- Box centered at body_height/2 so bottom is at z=0 -->
       <origin xyz="0 0 ${body_height/2}" rpy="0 0 0" />
-      <material name="grey">
-        <color rgba="0.6 0.6 0.6 0.8" />
-      </material>
+      <material name="grey"><color rgba="0.6 0.6 0.6 0.8" /></material>
     </visual>
     <collision>
@@ -81,40 +38,33 @@
     </collision>
   </link>
-  <!-- ============================================ -->
-  <!-- LEFT WHEEL                                  -->
-  <!-- ============================================ -->
+  <!-- ZED CAMERA -->
+  <joint name="base_to_camera_joint" type="fixed">
+    <parent link="base_link" />
+    <child link="zed_camera_link" />
+    <origin xyz="${camera_forward} 0 ${camera_height}" rpy="0 ${camera_tilt} 0" />
+  </joint>
+  <link name="zed_camera_link" />
+  <!-- LEFT WHEEL -->
   <joint name="left_wheel_joint" type="fixed">
     <parent link="base_link" />
     <child link="left_wheel" />
-    <!-- Wheel at ground level (z = wheel_radius), offset to left (+y) -->
-    <origin xyz="0 ${body_width/2+wheel_y_offset} 0" rpy="${-pi/2} 0 0" />
+    <origin xyz="0 ${body_width/2 + wheel_y_offset} 0" rpy="${-pi/2} 0 0" />
   </joint>
   <link name="left_wheel">
     <visual>
-      <geometry>
-        <cylinder radius="${wheel_radius}" length="${wheel_width}" />
-      </geometry>
-      <material name="dark_grey">
-        <color rgba="0.2 0.2 0.2 1.0" />
-      </material>
+      <geometry><cylinder radius="${wheel_radius}" length="${wheel_width}" /></geometry>
+      <material name="dark_grey"><color rgba="0.2 0.2 0.2 1.0" /></material>
     </visual>
   </link>
-  <!-- ============================================ -->
-  <!-- RIGHT WHEEL                                 -->
-  <!-- ============================================ -->
+  <!-- RIGHT WHEEL -->
   <joint name="right_wheel_joint" type="fixed">
     <parent link="base_link" />
     <child link="right_wheel" />
-    <!-- Wheel at ground level, offset to right (-y) -->
-    <origin xyz="0 ${-body_width/2-wheel_y_offset} 0" rpy="${-pi/2} 0 0" />
+    <origin xyz="0 ${-body_width/2 - wheel_y_offset} 0" rpy="${-pi/2} 0 0" />
   </joint>
   <link name="right_wheel">
     <visual>
-      <geometry>
-        <cylinder radius="${wheel_radius}" length="${wheel_width}" />
-      </geometry>
-      <material name="dark_grey">
-        <color rgba="0.2 0.2 0.2 1.0" />
-      </material>
+      <geometry><cylinder radius="${wheel_radius}" length="${wheel_width}" /></geometry>
+      <material name="dark_grey"><color rgba="0.2 0.2 0.2 1.0" /></material>
     </visual>
   </link>
