Commit message: fix: frame transforms

File: CODE/ros_ws/src/robot_bringup/urdf/robot.urdf.xacro (robot description, xacro)
@@ -5,8 +5,9 @@
     map → odom → base_link → zed_camera_link
     (node) (node)   (URDF)
-  Camera mounting (in base_link frame):
-    - 0.746m above base_link (Z)
-    - 0.174m forward of base_link center (X)
-    - 30° nose-down tilt (pitch = 0.523 rad)
+  Frame convention:
+    - base_link origin is at ground level (z=0)
+    - Wheel centers are at z=wheel_radius (0.05m), bottoms touch ground
+    - Body bottom face is at z=wheel_radius, sitting on top of axles
+    - Camera is camera_height (0.746m) above base_link, tilted 30° down
   ZED config: publish_tf: false, publish_map_tf: false
   odom_base_publisher handles all dynamic TFs.
@@ -14,11 +15,13 @@
 <robot xmlns:xacro="http://www.ros.org/wiki/xacro" name="material_transfer_robot">
   <xacro:property name="body_length" value="0.40" />
-  <xacro:property name="body_width"  value="0.30" />
+  <xacro:property name="body_width" value="0.30" />
   <xacro:property name="body_height" value="0.70" />
-  <xacro:property name="camera_height"  value="0.746" />
+  <xacro:property name="camera_height" value="0.746" />
+  <!-- from base_link origin -->
   <xacro:property name="camera_forward" value="0.174" />
-  <xacro:property name="camera_tilt"    value="0.523" />
-  <xacro:property name="wheel_radius"   value="0.075" />
-  <xacro:property name="wheel_width"    value="0.026" />
+  <xacro:property name="camera_tilt" value="0.523" />
+  <!-- 30° nose-down -->
+  <xacro:property name="wheel_radius" value="0.05" />
+  <xacro:property name="wheel_width" value="0.026" />
   <xacro:property name="wheel_y_offset" value="0.063" />
   <!-- BASE LINK -->
@@ -28,6 +31,9 @@
         <box size="${body_length} ${body_width} ${body_height}" />
       </geometry>
+      <!-- Bottom of box flush with axle, center at half height above -->
       <origin xyz="0 0 ${body_height/2}" rpy="0 0 0" />
-      <material name="grey"><color rgba="0.6 0.6 0.6 0.8" /></material>
+      <material name="grey">
+        <color rgba="0.6 0.6 0.6 0.8" />
+      </material>
     </visual>
     <collision>
@@ -38,12 +44,13 @@
     </collision>
   </link>
-  <!-- ZED CAMERA -->
+  <!-- ZED CAMERA — camera_height above base_link, tilted 30° nose-down -->
   <joint name="base_to_camera_joint" type="fixed">
     <parent link="base_link" />
     <child link="zed_camera_link" />
+    <!-- camera_height is measured from base_link origin, no wheel_radius needed here -->
     <origin xyz="${camera_forward} 0 ${camera_height}" rpy="0 ${camera_tilt} 0" />
   </joint>
   <link name="zed_camera_link" />
-  <!-- LEFT WHEEL -->
+  <!-- LEFT WHEEL — center at z=wheel_radius so bottom touches ground -->
   <joint name="left_wheel_joint" type="fixed">
     <parent link="base_link" />
@@ -53,9 +60,18 @@
   <link name="left_wheel">
     <visual>
-      <geometry><cylinder radius="${wheel_radius}" length="${wheel_width}" /></geometry>
-      <material name="dark_grey"><color rgba="0.2 0.2 0.2 1.0" /></material>
+      <geometry>
+        <cylinder radius="${wheel_radius}" length="${wheel_width}" />
+      </geometry>
+      <material name="dark_grey">
+        <color rgba="0.2 0.2 0.2 1.0" />
+      </material>
     </visual>
+    <collision>
+      <geometry>
+        <cylinder radius="${wheel_radius}" length="${wheel_width}" />
+      </geometry>
+    </collision>
   </link>
-  <!-- RIGHT WHEEL -->
+  <!-- RIGHT WHEEL — center at z=wheel_radius so bottom touches ground -->
   <joint name="right_wheel_joint" type="fixed">
     <parent link="base_link" />
@@ -65,7 +81,16 @@
   <link name="right_wheel">
     <visual>
-      <geometry><cylinder radius="${wheel_radius}" length="${wheel_width}" /></geometry>
-      <material name="dark_grey"><color rgba="0.2 0.2 0.2 1.0" /></material>
+      <geometry>
+        <cylinder radius="${wheel_radius}" length="${wheel_width}" />
+      </geometry>
+      <material name="dark_grey">
+        <color rgba="0.2 0.2 0.2 1.0" />
+      </material>
     </visual>
+    <collision>
+      <geometry>
+        <cylinder radius="${wheel_radius}" length="${wheel_width}" />
+      </geometry>
+    </collision>
   </link>
 </robot>

Commit message: fix: remap tf tree and delete odom base publisher

File: CODE/ros_ws/src/robot_bringup/urdf/robot.urdf.xacro (robot description, xacro)
@@ -2,14 +2,17 @@
 <!--
   robot.urdf.xacro
-  TF Tree (with odom_base_publisher node):
-    map → odom → base_link → zed_camera_link
-    (node) (node)   (URDF)
+  TF Tree (ZED-rooted, no odom_base_publisher):
+    map → odom → zed_left_camera_frame → zed_camera_link → base_link → left_wheel
+                                        → zed_imu_link              → right_wheel
+                                        → zed_right_camera_frame
+                                        → zed_camera_center
+                                        → (other ZED internal frames)
   Frame convention:
-    - base_link origin is at ground level (z=0)
-    - Wheel centers are at z=wheel_radius (0.05m), bottoms touch ground
-    - Body bottom face is at z=wheel_radius, sitting on top of axles
-    - Camera is camera_height (0.746m) above base_link, tilted 30° down
-  ZED config: publish_tf: false, publish_map_tf: false
-  odom_base_publisher handles all dynamic TFs.
+    - zed_camera_link is the ZED's gravity-aligned root (two_d_mode + set_gravity_as_origin)
+    - base_link hangs off zed_camera_link, offset back and down to ground level
+    - No tilt in the joint — ZED gravity alignment already levels the frame
+    - Wheel visuals are children of base_link as before
+  ZED config: publish_tf: true, two_d_mode: true, set_gravity_as_origin: true
+  No odom_base_publisher needed — ZED owns map→odom→zed_left_camera_frame→zed_camera_link
 -->
 <robot xmlns:xacro="http://www.ros.org/wiki/xacro" name="material_transfer_robot">
@@ -18,12 +21,21 @@
   <xacro:property name="body_height" value="0.70" />
   <xacro:property name="camera_height" value="0.746" />
-  <!-- from base_link origin -->
+  <!-- camera is this far above ground -->
   <xacro:property name="camera_forward" value="0.174" />
-  <xacro:property name="camera_tilt" value="0.523" />
-  <!-- 30° nose-down -->
+  <!-- camera is this far forward of robot center -->
   <xacro:property name="wheel_radius" value="0.05" />
   <xacro:property name="wheel_width" value="0.026" />
   <xacro:property name="wheel_y_offset" value="0.063" />
-  <!-- BASE LINK -->
+  <!-- ZED CAMERA LINK — root of URDF tree, owned by ZED SDK TF broadcaster -->
+  <!-- Declared here so robot_state_publisher knows it exists as a root -->
+  <link name="zed_camera_link" />
+  <!-- BASE LINK — child of zed_camera_link, offset back to robot center and down to ground -->
+  <joint name="camera_to_base_joint" type="fixed">
+    <parent link="zed_camera_link" />
+    <child link="base_link" />
+    <!-- Inverse of original mount offset: back by camera_forward, down by camera_height -->
+    <!-- No RPY — ZED gravity alignment (two_d_mode + set_gravity_as_origin) levels the frame -->
+    <origin xyz="${-camera_forward} 0 ${-camera_height}" rpy="0 0 0" />
+  </joint>
   <link name="base_link">
     <visual>
@@ -31,5 +43,5 @@
         <box size="${body_length} ${body_width} ${body_height}" />
       </geometry>
-      <!-- Bottom of box flush with axle, center at half height above -->
+      <!-- Body center is at half height above base_link origin (ground level) -->
       <origin xyz="0 0 ${body_height/2}" rpy="0 0 0" />
       <material name="grey">
@@ -44,13 +56,5 @@
     </collision>
   </link>
-  <!-- ZED CAMERA — camera_height above base_link, tilted 30° nose-down -->
-  <joint name="base_to_camera_joint" type="fixed">
-    <parent link="base_link" />
-    <child link="zed_camera_link" />
-    <!-- camera_height is measured from base_link origin, no wheel_radius needed here -->
-    <origin xyz="${camera_forward} 0 ${camera_height}" rpy="0 ${camera_tilt} 0" />
-  </joint>
-  <link name="zed_camera_link" />
-  <!-- LEFT WHEEL — center at z=wheel_radius so bottom touches ground -->
+  <!-- LEFT WHEEL -->
   <joint name="left_wheel_joint" type="fixed">
     <parent link="base_link" />
@@ -73,5 +77,5 @@
     </collision>
   </link>
-  <!-- RIGHT WHEEL — center at z=wheel_radius so bottom touches ground -->
+  <!-- RIGHT WHEEL -->
   <joint name="right_wheel_joint" type="fixed">
     <parent link="base_link" />

Commit message: fix: move block above zed

File: CODE/ros_ws/src/robot_bringup/urdf/robot.urdf.xacro (robot description, xacro)
@@ -36,5 +36,5 @@
     <!-- Inverse of original mount offset: back by camera_forward, down by camera_height -->
     <!-- No RPY — ZED gravity alignment (two_d_mode + set_gravity_as_origin) levels the frame -->
-    <origin xyz="${-camera_forward} 0 ${-camera_height}" rpy="0 0 0" />
+    <origin xyz="${camera_forward} 0 ${wheel_radius}" rpy="0 0 0" />
   </joint>
   <link name="base_link">

Commit message: fix: floor filtering

File: CODE/ros_ws/src/robot_bringup/urdf/robot.urdf.xacro (robot description, xacro)
@@ -17,61 +17,74 @@
 -->
 <robot xmlns:xacro="http://www.ros.org/wiki/xacro" name="material_transfer_robot">
-  <xacro:property name="body_length" value="0.40" />
-  <xacro:property name="body_width" value="0.30" />
-  <xacro:property name="body_height" value="0.70" />
-  <xacro:property name="camera_height" value="0.746" />
-  <!-- camera is this far above ground -->
-  <xacro:property name="camera_forward" value="0.174" />
-  <!-- camera is this far forward of robot center -->
-  <xacro:property name="wheel_radius" value="0.05" />
-  <xacro:property name="wheel_width" value="0.026" />
-  <xacro:property name="wheel_y_offset" value="0.063" />
+  <xacro:property name="body_length" value="0.40"/>
+  <xacro:property name="body_width" value="0.30"/>
+  <xacro:property name="body_height" value="0.70"/>
+  <xacro:property name="camera_height" value="0.746"/>
+  <xacro:property name="camera_forward" value="0.174"/>
+  <xacro:property name="camera_tilt" value="-0.5236"/>
+  <xacro:property name="wheel_radius" value="0.05"/>
+  <xacro:property name="wheel_width" value="0.026"/>
+  <xacro:property name="wheel_y_offset" value="0.063"/>
   <!-- ZED CAMERA LINK — root of URDF tree, owned by ZED SDK TF broadcaster -->
   <!-- Declared here so robot_state_publisher knows it exists as a root -->
-  <link name="zed_camera_link" />
-  <!-- BASE LINK — child of zed_camera_link, offset back to robot center and down to ground -->
+  <link name="zed_camera_link"/>
+  <!-- Camera mount frame: true physical pose (height + tilt) -->
+  <link name="camera_mount"/>
+  <joint name="zed_to_camera_mount" type="fixed">
+    <parent link="zed_camera_link"/>
+    <child link="camera_mount"/>
+    <!-- Raise by camera_height and apply tilt (no forward offset here) -->
+    <origin xyz="0 0 ${camera_height}" rpy="0 ${camera_tilt} 0"/>
+  </joint>
+  <!-- BASE LINK — upright, at robot center, raised by wheel_radius -->
   <joint name="camera_to_base_joint" type="fixed">
-    <parent link="zed_camera_link" />
-    <child link="base_link" />
-    <!-- Inverse of original mount offset: back by camera_forward, down by camera_height -->
-    <!-- No RPY — ZED gravity alignment (two_d_mode + set_gravity_as_origin) levels the frame -->
-    <origin xyz="${camera_forward} 0 ${wheel_radius}" rpy="0 0 0" />
+    <parent link="zed_camera_link"/>
+    <child link="base_link"/>
+    <!-- zed_camera_link is at ground, base_link at wheel_radius above ground -->
+    <origin xyz="${-camera_forward} 0 ${wheel_radius}" rpy="0 0 0"/>
+  </joint>
+  <!-- Ground frame at floor level -->
+  <link name="ground"/>
+  <joint name="base_to_ground" type="fixed">
+    <parent link="base_link"/>
+    <child link="ground"/>
+    <origin xyz="0 0 ${-wheel_radius}" rpy="0 0 0"/>
   </joint>
   <link name="base_link">
     <visual>
       <geometry>
-        <box size="${body_length} ${body_width} ${body_height}" />
+        <box size="${body_length} ${body_width} ${body_height}"/>
       </geometry>
       <!-- Body center is at half height above base_link origin (ground level) -->
-      <origin xyz="0 0 ${body_height/2}" rpy="0 0 0" />
+      <origin xyz="0 0 ${body_height/2}" rpy="0 0 0"/>
       <material name="grey">
-        <color rgba="0.6 0.6 0.6 0.8" />
+        <color rgba="0.6 0.6 0.6 0.8"/>
       </material>
     </visual>
     <collision>
       <geometry>
-        <box size="${body_length} ${body_width} ${body_height}" />
+        <box size="${body_length} ${body_width} ${body_height}"/>
       </geometry>
-      <origin xyz="0 0 ${body_height/2}" rpy="0 0 0" />
+      <origin xyz="0 0 ${body_height/2}" rpy="0 0 0"/>
     </collision>
   </link>
   <!-- LEFT WHEEL -->
   <joint name="left_wheel_joint" type="fixed">
-    <parent link="base_link" />
-    <child link="left_wheel" />
-    <origin xyz="0 ${body_width/2 + wheel_y_offset} 0" rpy="${-pi/2} 0 0" />
+    <parent link="base_link"/>
+    <child link="left_wheel"/>
+    <origin xyz="0 ${body_width/2 + wheel_y_offset} 0" rpy="${-pi/2} 0 0"/>
   </joint>
   <link name="left_wheel">
     <visual>
       <geometry>
-        <cylinder radius="${wheel_radius}" length="${wheel_width}" />
+        <cylinder radius="${wheel_radius}" length="${wheel_width}"/>
       </geometry>
       <material name="dark_grey">
-        <color rgba="0.2 0.2 0.2 1.0" />
+        <color rgba="0.2 0.2 0.2 1.0"/>
       </material>
     </visual>
     <collision>
       <geometry>
-        <cylinder radius="${wheel_radius}" length="${wheel_width}" />
+        <cylinder radius="${wheel_radius}" length="${wheel_width}"/>
       </geometry>
     </collision>
@@ -79,20 +92,20 @@
   <!-- RIGHT WHEEL -->
   <joint name="right_wheel_joint" type="fixed">
-    <parent link="base_link" />
-    <child link="right_wheel" />
-    <origin xyz="0 ${-body_width/2 - wheel_y_offset} 0" rpy="${-pi/2} 0 0" />
+    <parent link="base_link"/>
+    <child link="right_wheel"/>
+    <origin xyz="0 ${-body_width/2 - wheel_y_offset} 0" rpy="${-pi/2} 0 0"/>
   </joint>
   <link name="right_wheel">
     <visual>
       <geometry>
-        <cylinder radius="${wheel_radius}" length="${wheel_width}" />
+        <cylinder radius="${wheel_radius}" length="${wheel_width}"/>
       </geometry>
       <material name="dark_grey">
-        <color rgba="0.2 0.2 0.2 1.0" />
+        <color rgba="0.2 0.2 0.2 1.0"/>
       </material>
     </visual>
     <collision>
       <geometry>
-        <cylinder radius="${wheel_radius}" length="${wheel_width}" />
+        <cylinder radius="${wheel_radius}" length="${wheel_width}"/>
       </geometry>
     </collision>

Commit message: fix: camera tilt

File: CODE/ros_ws/src/robot_bringup/urdf/robot.urdf.xacro (robot description, xacro)
@@ -22,5 +22,5 @@
   <xacro:property name="camera_height" value="0.746"/>
   <xacro:property name="camera_forward" value="0.174"/>
-  <xacro:property name="camera_tilt" value="-0.5236"/>
+  <xacro:property name="camera_tilt" value="0.5236"/>
   <xacro:property name="wheel_radius" value="0.05"/>
   <xacro:property name="wheel_width" value="0.026"/>

Commit message: fix: camera mount child of base link

File: CODE/ros_ws/src/robot_bringup/urdf/robot.urdf.xacro (robot description, xacro)
@@ -17,74 +17,72 @@
 -->
 <robot xmlns:xacro="http://www.ros.org/wiki/xacro" name="material_transfer_robot">
-  <xacro:property name="body_length" value="0.40"/>
-  <xacro:property name="body_width" value="0.30"/>
-  <xacro:property name="body_height" value="0.70"/>
-  <xacro:property name="camera_height" value="0.746"/>
-  <xacro:property name="camera_forward" value="0.174"/>
-  <xacro:property name="camera_tilt" value="0.5236"/>
-  <xacro:property name="wheel_radius" value="0.05"/>
-  <xacro:property name="wheel_width" value="0.026"/>
-  <xacro:property name="wheel_y_offset" value="0.063"/>
+  <xacro:property name="body_length" value="0.40" />
+  <xacro:property name="body_width" value="0.30" />
+  <xacro:property name="body_height" value="0.70" />
+  <xacro:property name="camera_height" value="0.746" />
+  <xacro:property name="camera_forward" value="0.174" />
+  <xacro:property name="camera_tilt" value="0.5236" />
+  <xacro:property name="wheel_radius" value="0.05" />
+  <xacro:property name="wheel_width" value="0.026" />
+  <xacro:property name="wheel_y_offset" value="0.063" />
   <!-- ZED CAMERA LINK — root of URDF tree, owned by ZED SDK TF broadcaster -->
   <!-- Declared here so robot_state_publisher knows it exists as a root -->
-  <link name="zed_camera_link"/>
+  <!-- BASE LINK — upright, at robot center, raised by wheel_radius -->
+  <link name="zed_camera_link" />
+  <joint name="camera_to_base_joint" type="fixed">
+    <parent link="zed_camera_link" />
+    <child link="base_link" />
+    <origin xyz="${-camera_forward} 0 ${wheel_radius}" rpy="0 0 0" />
+  </joint>
   <!-- Camera mount frame: true physical pose (height + tilt) -->
-  <link name="camera_mount"/>
+  <link name="camera_mount" />
   <joint name="zed_to_camera_mount" type="fixed">
-    <parent link="zed_camera_link"/>
-    <child link="camera_mount"/>
-    <!-- Raise by camera_height and apply tilt (no forward offset here) -->
-    <origin xyz="0 0 ${camera_height}" rpy="0 ${camera_tilt} 0"/>
-  </joint>
-  <!-- BASE LINK — upright, at robot center, raised by wheel_radius -->
-  <joint name="camera_to_base_joint" type="fixed">
-    <parent link="zed_camera_link"/>
-    <child link="base_link"/>
-    <!-- zed_camera_link is at ground, base_link at wheel_radius above ground -->
-    <origin xyz="${-camera_forward} 0 ${wheel_radius}" rpy="0 0 0"/>
+    <parent link="base_link" />
+    <child link="camera_mount" />
+    <origin xyz="${camera_forward} 0 ${camera_height}" rpy="0 ${camera_tilt} 0" />
   </joint>
   <!-- Ground frame at floor level -->
-  <link name="ground"/>
+  <link name="ground" />
   <joint name="base_to_ground" type="fixed">
-    <parent link="base_link"/>
-    <child link="ground"/>
-    <origin xyz="0 0 ${-wheel_radius}" rpy="0 0 0"/>
+    <parent link="base_link" />
+    <child link="ground" />
+    <origin xyz="0 0 ${-wheel_radius}" rpy="0 0 0" />
   </joint>
   <link name="base_link">
     <visual>
       <geometry>
-        <box size="${body_length} ${body_width} ${body_height}"/>
+        <box size="${body_length} ${body_width} ${body_height}" />
       </geometry>
       <!-- Body center is at half height above base_link origin (ground level) -->
-      <origin xyz="0 0 ${body_height/2}" rpy="0 0 0"/>
+      <origin xyz="0 0 ${body_height/2}" rpy="0 0 0" />
       <material name="grey">
-        <color rgba="0.6 0.6 0.6 0.8"/>
+        <color rgba="0.6 0.6 0.6 0.8" />
       </material>
     </visual>
     <collision>
       <geometry>
-        <box size="${body_length} ${body_width} ${body_height}"/>
+        <box size="${body_length} ${body_width} ${body_height}" />
       </geometry>
-      <origin xyz="0 0 ${body_height/2}" rpy="0 0 0"/>
+      <origin xyz="0 0 ${body_height/2}" rpy="0 0 0" />
     </collision>
   </link>
   <!-- LEFT WHEEL -->
   <joint name="left_wheel_joint" type="fixed">
-    <parent link="base_link"/>
-    <child link="left_wheel"/>
-    <origin xyz="0 ${body_width/2 + wheel_y_offset} 0" rpy="${-pi/2} 0 0"/>
+    <parent link="base_link" />
+    <child link="left_wheel" />
+    <origin xyz="0 ${body_width/2 + wheel_y_offset} 0" rpy="${-pi/2} 0 0" />
   </joint>
   <link name="left_wheel">
     <visual>
       <geometry>
-        <cylinder radius="${wheel_radius}" length="${wheel_width}"/>
+        <cylinder radius="${wheel_radius}" length="${wheel_width}" />
       </geometry>
       <material name="dark_grey">
-        <color rgba="0.2 0.2 0.2 1.0"/>
+        <color rgba="0.2 0.2 0.2 1.0" />
       </material>
     </visual>
     <collision>
       <geometry>
-        <cylinder radius="${wheel_radius}" length="${wheel_width}"/>
+        <cylinder radius="${wheel_radius}" length="${wheel_width}" />
       </geometry>
     </collision>
@@ -92,20 +90,20 @@
   <!-- RIGHT WHEEL -->
   <joint name="right_wheel_joint" type="fixed">
-    <parent link="base_link"/>
-    <child link="right_wheel"/>
-    <origin xyz="0 ${-body_width/2 - wheel_y_offset} 0" rpy="${-pi/2} 0 0"/>
+    <parent link="base_link" />
+    <child link="right_wheel" />
+    <origin xyz="0 ${-body_width/2 - wheel_y_offset} 0" rpy="${-pi/2} 0 0" />
   </joint>
   <link name="right_wheel">
     <visual>
       <geometry>
-        <cylinder radius="${wheel_radius}" length="${wheel_width}"/>
+        <cylinder radius="${wheel_radius}" length="${wheel_width}" />
       </geometry>
       <material name="dark_grey">
-        <color rgba="0.2 0.2 0.2 1.0"/>
+        <color rgba="0.2 0.2 0.2 1.0" />
       </material>
     </visual>
     <collision>
       <geometry>
-        <cylinder radius="${wheel_radius}" length="${wheel_width}"/>
+        <cylinder radius="${wheel_radius}" length="${wheel_width}" />
       </geometry>
     </collision>
