Commit message: fix: update cam angle

File: CODE/ros_ws/src/robot_bringup/urdf/robot.urdf.xacro (robot description, xacro)
@@ -17,72 +17,72 @@
 -->
 <robot xmlns:xacro="http://www.ros.org/wiki/xacro" name="material_transfer_robot">
-  <xacro:property name="body_length" value="0.40" />
-  <xacro:property name="body_width" value="0.30" />
-  <xacro:property name="body_height" value="0.70" />
-  <xacro:property name="camera_height" value="0.746" />
-  <xacro:property name="camera_forward" value="0.174" />
-  <xacro:property name="camera_tilt" value="0.5236" />
-  <xacro:property name="wheel_radius" value="0.05" />
-  <xacro:property name="wheel_width" value="0.026" />
-  <xacro:property name="wheel_y_offset" value="0.063" />
+  <xacro:property name="body_length" value="0.40"/>
+  <xacro:property name="body_width" value="0.30"/>
+  <xacro:property name="body_height" value="0.70"/>
+  <xacro:property name="camera_height" value="0.746"/>
+  <xacro:property name="camera_forward" value="0.174"/>
+  <xacro:property name="camera_tilt" value="0.319"/>
+  <xacro:property name="wheel_radius" value="0.05"/>
+  <xacro:property name="wheel_width" value="0.026"/>
+  <xacro:property name="wheel_y_offset" value="0.063"/>
   <!-- ZED CAMERA LINK — root of URDF tree, owned by ZED SDK TF broadcaster -->
   <!-- Declared here so robot_state_publisher knows it exists as a root -->
   <!-- BASE LINK — upright, at robot center, raised by wheel_radius -->
-  <link name="zed_camera_link" />
+  <link name="zed_camera_link"/>
   <joint name="camera_to_base_joint" type="fixed">
-    <parent link="zed_camera_link" />
-    <child link="base_link" />
-    <origin xyz="${-camera_forward} 0 ${wheel_radius}" rpy="0 0 0" />
+    <parent link="zed_camera_link"/>
+    <child link="base_link"/>
+    <origin xyz="${-camera_forward} 0 ${wheel_radius}" rpy="0 0 0"/>
   </joint>
   <!-- Camera mount frame: true physical pose (height + tilt) -->
-  <link name="camera_mount" />
+  <link name="camera_mount"/>
   <joint name="zed_to_camera_mount" type="fixed">
-    <parent link="base_link" />
-    <child link="camera_mount" />
-    <origin xyz="${camera_forward} 0 ${camera_height}" rpy="0 ${camera_tilt} 0" />
+    <parent link="base_link"/>
+    <child link="camera_mount"/>
+    <origin xyz="${camera_forward} 0 ${camera_height}" rpy="0 ${camera_tilt} 0"/>
   </joint>
   <!-- Ground frame at floor level -->
-  <link name="ground" />
+  <link name="ground"/>
   <joint name="base_to_ground" type="fixed">
-    <parent link="base_link" />
-    <child link="ground" />
-    <origin xyz="0 0 ${-wheel_radius}" rpy="0 0 0" />
+    <parent link="base_link"/>
+    <child link="ground"/>
+    <origin xyz="0 0 ${-wheel_radius}" rpy="0 0 0"/>
   </joint>
   <link name="base_link">
     <visual>
       <geometry>
-        <box size="${body_length} ${body_width} ${body_height}" />
+        <box size="${body_length} ${body_width} ${body_height}"/>
       </geometry>
       <!-- Body center is at half height above base_link origin (ground level) -->
-      <origin xyz="0 0 ${body_height/2}" rpy="0 0 0" />
+      <origin xyz="0 0 ${body_height/2}" rpy="0 0 0"/>
       <material name="grey">
-        <color rgba="0.6 0.6 0.6 0.8" />
+        <color rgba="0.6 0.6 0.6 0.8"/>
       </material>
     </visual>
     <collision>
       <geometry>
-        <box size="${body_length} ${body_width} ${body_height}" />
+        <box size="${body_length} ${body_width} ${body_height}"/>
       </geometry>
-      <origin xyz="0 0 ${body_height/2}" rpy="0 0 0" />
+      <origin xyz="0 0 ${body_height/2}" rpy="0 0 0"/>
     </collision>
   </link>
   <!-- LEFT WHEEL -->
   <joint name="left_wheel_joint" type="fixed">
-    <parent link="base_link" />
-    <child link="left_wheel" />
-    <origin xyz="0 ${body_width/2 + wheel_y_offset} 0" rpy="${-pi/2} 0 0" />
+    <parent link="base_link"/>
+    <child link="left_wheel"/>
+    <origin xyz="0 ${body_width/2 + wheel_y_offset} 0" rpy="${-pi/2} 0 0"/>
   </joint>
   <link name="left_wheel">
     <visual>
       <geometry>
-        <cylinder radius="${wheel_radius}" length="${wheel_width}" />
+        <cylinder radius="${wheel_radius}" length="${wheel_width}"/>
       </geometry>
       <material name="dark_grey">
-        <color rgba="0.2 0.2 0.2 1.0" />
+        <color rgba="0.2 0.2 0.2 1.0"/>
       </material>
     </visual>
     <collision>
       <geometry>
-        <cylinder radius="${wheel_radius}" length="${wheel_width}" />
+        <cylinder radius="${wheel_radius}" length="${wheel_width}"/>
       </geometry>
     </collision>
@@ -90,20 +90,20 @@
   <!-- RIGHT WHEEL -->
   <joint name="right_wheel_joint" type="fixed">
-    <parent link="base_link" />
-    <child link="right_wheel" />
-    <origin xyz="0 ${-body_width/2 - wheel_y_offset} 0" rpy="${-pi/2} 0 0" />
+    <parent link="base_link"/>
+    <child link="right_wheel"/>
+    <origin xyz="0 ${-body_width/2 - wheel_y_offset} 0" rpy="${-pi/2} 0 0"/>
   </joint>
   <link name="right_wheel">
     <visual>
       <geometry>
-        <cylinder radius="${wheel_radius}" length="${wheel_width}" />
+        <cylinder radius="${wheel_radius}" length="${wheel_width}"/>
       </geometry>
       <material name="dark_grey">
-        <color rgba="0.2 0.2 0.2 1.0" />
+        <color rgba="0.2 0.2 0.2 1.0"/>
       </material>
     </visual>
     <collision>
       <geometry>
-        <cylinder radius="${wheel_radius}" length="${wheel_width}" />
+        <cylinder radius="${wheel_radius}" length="${wheel_width}"/>
       </geometry>
     </collision>

Commit message: fix: update cam tilt

File: CODE/ros_ws/src/robot_bringup/urdf/robot.urdf.xacro (robot description, xacro)
@@ -17,72 +17,72 @@
 -->
 <robot xmlns:xacro="http://www.ros.org/wiki/xacro" name="material_transfer_robot">
-  <xacro:property name="body_length" value="0.40"/>
-  <xacro:property name="body_width" value="0.30"/>
-  <xacro:property name="body_height" value="0.70"/>
-  <xacro:property name="camera_height" value="0.746"/>
-  <xacro:property name="camera_forward" value="0.174"/>
-  <xacro:property name="camera_tilt" value="0.319"/>
-  <xacro:property name="wheel_radius" value="0.05"/>
-  <xacro:property name="wheel_width" value="0.026"/>
-  <xacro:property name="wheel_y_offset" value="0.063"/>
+  <xacro:property name="body_length" value="0.40" />
+  <xacro:property name="body_width" value="0.30" />
+  <xacro:property name="body_height" value="0.70" />
+  <xacro:property name="camera_height" value="0.746" />
+  <xacro:property name="camera_forward" value="0.174" />
+  <xacro:property name="camera_tilt" value="0.258" />
+  <xacro:property name="wheel_radius" value="0.05" />
+  <xacro:property name="wheel_width" value="0.026" />
+  <xacro:property name="wheel_y_offset" value="0.063" />
   <!-- ZED CAMERA LINK — root of URDF tree, owned by ZED SDK TF broadcaster -->
   <!-- Declared here so robot_state_publisher knows it exists as a root -->
   <!-- BASE LINK — upright, at robot center, raised by wheel_radius -->
-  <link name="zed_camera_link"/>
+  <link name="zed_camera_link" />
   <joint name="camera_to_base_joint" type="fixed">
-    <parent link="zed_camera_link"/>
-    <child link="base_link"/>
-    <origin xyz="${-camera_forward} 0 ${wheel_radius}" rpy="0 0 0"/>
+    <parent link="zed_camera_link" />
+    <child link="base_link" />
+    <origin xyz="${-camera_forward} 0 ${wheel_radius}" rpy="0 0 0" />
   </joint>
   <!-- Camera mount frame: true physical pose (height + tilt) -->
-  <link name="camera_mount"/>
+  <link name="camera_mount" />
   <joint name="zed_to_camera_mount" type="fixed">
-    <parent link="base_link"/>
-    <child link="camera_mount"/>
-    <origin xyz="${camera_forward} 0 ${camera_height}" rpy="0 ${camera_tilt} 0"/>
+    <parent link="base_link" />
+    <child link="camera_mount" />
+    <origin xyz="${camera_forward} 0 ${camera_height}" rpy="0 ${camera_tilt} 0" />
   </joint>
   <!-- Ground frame at floor level -->
-  <link name="ground"/>
+  <link name="ground" />
   <joint name="base_to_ground" type="fixed">
-    <parent link="base_link"/>
-    <child link="ground"/>
-    <origin xyz="0 0 ${-wheel_radius}" rpy="0 0 0"/>
+    <parent link="base_link" />
+    <child link="ground" />
+    <origin xyz="0 0 ${-wheel_radius}" rpy="0 0 0" />
   </joint>
   <link name="base_link">
     <visual>
       <geometry>
-        <box size="${body_length} ${body_width} ${body_height}"/>
+        <box size="${body_length} ${body_width} ${body_height}" />
       </geometry>
       <!-- Body center is at half height above base_link origin (ground level) -->
-      <origin xyz="0 0 ${body_height/2}" rpy="0 0 0"/>
+      <origin xyz="0 0 ${body_height/2}" rpy="0 0 0" />
       <material name="grey">
-        <color rgba="0.6 0.6 0.6 0.8"/>
+        <color rgba="0.6 0.6 0.6 0.8" />
       </material>
     </visual>
     <collision>
       <geometry>
-        <box size="${body_length} ${body_width} ${body_height}"/>
+        <box size="${body_length} ${body_width} ${body_height}" />
       </geometry>
-      <origin xyz="0 0 ${body_height/2}" rpy="0 0 0"/>
+      <origin xyz="0 0 ${body_height/2}" rpy="0 0 0" />
     </collision>
   </link>
   <!-- LEFT WHEEL -->
   <joint name="left_wheel_joint" type="fixed">
-    <parent link="base_link"/>
-    <child link="left_wheel"/>
-    <origin xyz="0 ${body_width/2 + wheel_y_offset} 0" rpy="${-pi/2} 0 0"/>
+    <parent link="base_link" />
+    <child link="left_wheel" />
+    <origin xyz="0 ${body_width/2 + wheel_y_offset} 0" rpy="${-pi/2} 0 0" />
   </joint>
   <link name="left_wheel">
     <visual>
       <geometry>
-        <cylinder radius="${wheel_radius}" length="${wheel_width}"/>
+        <cylinder radius="${wheel_radius}" length="${wheel_width}" />
       </geometry>
       <material name="dark_grey">
-        <color rgba="0.2 0.2 0.2 1.0"/>
+        <color rgba="0.2 0.2 0.2 1.0" />
       </material>
     </visual>
     <collision>
       <geometry>
-        <cylinder radius="${wheel_radius}" length="${wheel_width}"/>
+        <cylinder radius="${wheel_radius}" length="${wheel_width}" />
       </geometry>
     </collision>
@@ -90,20 +90,20 @@
   <!-- RIGHT WHEEL -->
   <joint name="right_wheel_joint" type="fixed">
-    <parent link="base_link"/>
-    <child link="right_wheel"/>
-    <origin xyz="0 ${-body_width/2 - wheel_y_offset} 0" rpy="${-pi/2} 0 0"/>
+    <parent link="base_link" />
+    <child link="right_wheel" />
+    <origin xyz="0 ${-body_width/2 - wheel_y_offset} 0" rpy="${-pi/2} 0 0" />
   </joint>
   <link name="right_wheel">
     <visual>
       <geometry>
-        <cylinder radius="${wheel_radius}" length="${wheel_width}"/>
+        <cylinder radius="${wheel_radius}" length="${wheel_width}" />
       </geometry>
       <material name="dark_grey">
-        <color rgba="0.2 0.2 0.2 1.0"/>
+        <color rgba="0.2 0.2 0.2 1.0" />
       </material>
     </visual>
     <collision>
       <geometry>
-        <cylinder radius="${wheel_radius}" length="${wheel_width}"/>
+        <cylinder radius="${wheel_radius}" length="${wheel_width}" />
       </geometry>
     </collision>
